File: KiCAD/RC-two-wheeler.kicad_pcb (KiCad board)
At the start: 2 copper layers, 50 x 50 mm, 15 parts, among them J1 Conn_01x03_Male, J2 Conn_01x03_Male, J3 Conn_01x03_Male, J4 Conn_01x05_Male, SW1 SW_DPDT_x2, U1 NRF24L01_Breakout

Commit message: Added 2 led and made DRC
Parts:
- added D1: LED, LED_SMD:LED_0603_1608Metric_Pad1.05x0.95mm_HandSolder, F.Cu at (87.5, 77.0)
- added D2: LED, LED_SMD:LED_0603_1608Metric_Pad1.05x0.95mm_HandSolder, F.Cu at (87.5, 79.0)
- added R6: R, Resistor_SMD:R_0603_1608Metric_Pad1.05x0.95mm_HandSolder, F.Cu at (126.7, 95.5)
- added R7: R, Resistor_SMD:R_0603_1608Metric_Pad1.05x0.95mm_HandSolder, F.Cu at (126.7, 97.0)
- added R8: R, Resistor_SMD:R_0603_1608Metric_Pad1.05x0.95mm_HandSolder, F.Cu at (91.0, 77.0)
- added R9: R, Resistor_SMD:R_0603_1608Metric_Pad1.05x0.95mm_HandSolder, F.Cu at (91.0, 79.0)
- added REF**: MountingHole_3.2mm_M3, MountingHole:MountingHole_3.2mm_M3, F.Cu at (95.0, 120.0)
- added REF**: MountingHole_3.2mm_M3, MountingHole:MountingHole_3.2mm_M3, F.Cu at (110.0, 80.0)
- added REF**: MountingHole_3.2mm_M3, MountingHole:MountingHole_3.2mm_M3, F.Cu at (130.0, 120.0)
- turned SW1 to 270 degrees
Connections:
- A1 pad 22: Net-(A1-Pad22) -> /batVoltage
- J1 pad 1: GND -> Net-(J1-Pad1)
- J1 pad 3: Net-(J1-Pad3) -> GND
- SW1 pad 1: Net-(J1-Pad3) -> Net-(J1-Pad1)
Routing:
- net +3V3: track 10.4 -> 52.2 mm, vias 0 -> 2
- net Net-(J1-Pad1): track 0.00 -> 25.7 mm
- net Net-(A1-Pad6): track 0.00 -> 25.5 mm, vias 0 -> 1
- net Net-(A1-Pad7): track 0.00 -> 24.0 mm, vias 0 -> 1
- net Net-(J1-Pad3): track 19.7 -> 0.00 mm
- net /batVoltage: track 0.00 -> 11.5 mm
- net GND: track 4.12 -> 11.6 mm, vias 3 -> 5
- net Net-(D2-Pad1): track 0.00 -> 1.78 mm
- net Net-(D1-Pad1): track 0.00 -> 1.78 mm
- net Net-(SW1-Pad3): track 5.50 -> 6.15 mm

Commit message: Updated rev date to 20200209
Other:
- board text added: "RC Two Wheeler 2020-02-09 rev 1"
- board text removed: "RC Two Wheeler 2020-02-05 rev 1"
Changed lines of the file:
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@@
       (psnegative false)
       (psa4output false)
-      (plotreference true)
-      (plotvalue true)
+      (plotreference false)
+      (plotvalue false)
       (plotinvisibletext false)
       (padsonsilk false)
@@
       (outputformat 1)
       (mirror false)
-      (drillshape 1)
+      (drillshape 0)
       (scaleselection 1)
-      (outputdirectory ""))
+      (outputdirectory "Gerber/"))
   )
   (net 0 "")
@@
     (effects (font (size 1.2 1.2) (thickness 0.2)))
   )
-  (gr_text "RC Two Wheeler\n2020-02-05\nrev 1" (at 127.25 102) (layer F.SilkS)
+  (gr_text "RC Two Wheeler\n2020-02-09\nrev 1" (at 127.25 102) (layer F.SilkS)
     (effects (font (size 1.2 1.2) (thickness 0.2)))
   )
